File: NTC/Main.kicad_pcb (KiCad board)
At the start: 2 copper layers, 307.3 x 144.8 mm, 252 parts, among them Q1 MPSA42, Q10 MPSA42, Q11 MPSA42, Q12 MPSA42, Q13 MPSA42, Q14 MPSA42, Q15 MPSA42, Q16 MPSA42, Q17 MPSA42, Q18 MPSA42, Q19 MPSA42, Q2 MPSA42, Q20 MPSA42, Q21 MPSA42, Q22 MPSA42, Q23 MPSA42, Q24 MPSA42, Q25 MPSA42, Q26 MPSA42, Q27 MPSA42, Q28 MPSA42, Q29 MPSA42, Q3 MPSA42, Q30 MPSA42, Q31 MPSA42, Q32 MPSA42, Q33 MPSA42, Q34 MPSA42, Q35 MPSA42, Q36 MPSA42, Q37 MPSA42, Q38 MPSA42, Q39 MPSA42, Q4 MPSA42, Q40 MPSA42, Q41 MPSA42, Q42 MPSA42, Q43 MPSA42, Q44 MPSA42, Q45 MPSA42, Q46 MPSA42, Q47 MPSA42, Q48 MPSA42, Q49 MPSA42, Q5 MPSA42, Q50 MPSA42, Q51 MPSA42, Q52 MPSA42, Q53 MPSA42, Q54 MPSA42, Q55 MPSA42, Q56 MPSA42, Q57 MPSA42, Q58 MPSA42, Q59 MPSA42, Q6 MPSA42, Q60 MPSA42, Q61 MPSA42, Q62 MPSA42, Q63 MPSA42, Q64 MPSA42, Q65 MPSA42, Q66 MPSA42, Q67 MPSA42, Q68 MPSA42, Q69 MPSA42, Q7 MPSA42, Q70 MPSA42, Q8 MPSA42, Q9 MPSA42, U1 TDN_5-0911WISM, X1 Barrel_Jack_Switch, X10 Conn_01x06_Socket, X11 Conn_01x04_Socket, X12 Conn_01x06_Socket, X13 Conn_01x06_Socket, X14 Conn_01x06_Socket, X15 Conn_01x06_Socket, X16 Conn_01x06_Socket, X17 Conn_01x06_Socket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

Commit message: Added QR
Other:
- board text removed: "MMXXIV"
