File: NTC/Main.kicad_pcb (KiCad board)
At the start: 2 copper layers, 307.3 x 144.8 mm, 252 parts, among them Q1 MPSA42, Q10 MPSA42, Q11 MPSA42, Q12 MPSA42, Q13 MPSA42, Q14 MPSA42, Q15 MPSA42, Q16 MPSA42, Q17 MPSA42, Q18 MPSA42, Q19 MPSA42, Q2 MPSA42, Q20 MPSA42, Q21 MPSA42, Q22 MPSA42, Q23 MPSA42, Q24 MPSA42, Q25 MPSA42, Q26 MPSA42, Q27 MPSA42, Q28 MPSA42, Q29 MPSA42, Q3 MPSA42, Q30 MPSA42, Q31 MPSA42, Q32 MPSA42, Q33 MPSA42, Q34 MPSA42, Q35 MPSA42, Q36 MPSA42, Q37 MPSA42, Q38 MPSA42, Q39 MPSA42, Q4 MPSA42, Q40 MPSA42, Q41 MPSA42, Q42 MPSA42, Q43 MPSA42, Q44 MPSA42, Q45 MPSA42, Q46 MPSA42, Q47 MPSA42, Q48 MPSA42, Q49 MPSA42, Q5 MPSA42, Q50 MPSA42, Q51 MPSA42, Q52 MPSA42, Q53 MPSA42, Q54 MPSA42, Q55 MPSA42, Q56 MPSA42, Q57 MPSA42, Q58 MPSA42, Q59 MPSA42, Q6 MPSA42, Q60 MPSA42, Q61 MPSA42, Q62 MPSA42, Q63 MPSA42, Q64 MPSA42, Q65 MPSA42, Q66 MPSA42, Q67 MPSA42, Q68 MPSA42, Q69 MPSA42, Q7 MPSA42, Q70 MPSA42, Q8 MPSA42, Q9 MPSA42, U1 TDN_5-0911WISM, X1 Barrel_Jack_Switch, X10 Conn_01x06_Socket, X11 Conn_01x04_Socket, X12 Conn_01x06_Socket, X13 Conn_01x06_Socket, X14 Conn_01x06_Socket, X15 Conn_01x06_Socket, X16 Conn_01x06_Socket, X17 Conn_01x06_Socket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

Commit message: Added alternative DC/DC converter and Tube schematic
Parts:
- added U2: R-78E5.0-1.0, Nixie:DCDC_12V-5V-5W, F.Cu at (48.3, 91.4)
- moved E1 5.08 mm to (45.7, 104.1)
Routing:
- net Net-(U1-+VIN): track 46.5 -> 54.1 mm
- net Net-(U1-+VOUT): track 73.4 -> 80.3 mm
- net Net-(U1-ON/OFF): track 6.13 -> 2.54 mm
- net /Tube_1-2/GND: track 1993.6 -> 1995.7 mm
- net /Tube_1-2/3V3: track 954.8 -> 956.3 mm

Commit message: Changed to 14pin socket
Parts:
- removed the X10 at (119.4, 94.0)
- removed the X13 at (175.3, 94.0)
- removed the X15 at (200.7, 94.0)
- removed X17, X19: Conn_01x06_Socket, Nixie:Pinbar_1-6-f-b
- removed the X9 at (119.4, 76.2)
- X10: renamed from X12; footprint Nixie:Pinbar_1-6-f-a -> Nixie:Pinbar_4-14-f
- X11: renamed from X14; footprint Nixie:Pinbar_1-6-f-a -> Nixie:Pinbar_4-14-f
- X12: renamed from X16; footprint Nixie:Pinbar_1-6-f-a -> Nixie:Pinbar_4-14-f
- X13: renamed from X18; footprint Nixie:Pinbar_1-6-f-a -> Nixie:Pinbar_4-14-f
- X7: footprint Nixie:Pinbar_1-6-f-a -> Nixie:Pinbar_4-14-f
- X8: footprint Nixie:Pinbar_1-6-f-b -> Nixie:Pinbar_4-14-f
- moved X8 67.5 mm to (157.5, 116.8)
- moved X12 63.1 mm to (304.8, 116.8)
- moved X13 63.1 mm to (330.2, 116.8)
- moved X10 59.3 mm to (218.4, 116.8)
- moved X11 59.3 mm to (243.8, 116.8)
- moved REF** 56.8 mm to (364.5, 47.0)
- moved Q63 55.7 mm to (332.7, 149.9)
- moved R92 55.7 mm to (340.4, 149.9)
- moved X7 55.7 mm to (132.1, 116.8)
- moved Q65 55.7 mm to (337.8, 139.7)
- moved Q66 55.7 mm to (340.4, 134.6)
- moved Q68 55.7 mm to (345.4, 124.5)
- moved R85 55.7 mm to (358.1, 91.4)
- moved R91 55.7 mm to (337.8, 154.9)
- moved R94 55.7 mm to (345.4, 139.7)
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- renumbered X20 to X14, X21 to X15, X11 to X9
Connections:
- R1 pad 2: Net-(X7-Pin_3) -> Net-(X7-Pin_4)
- R16 pad 2: Net-(X9-Pin_3) (its old number) -> Net-(X8-Pin_4)
- R21 pad 1: Net-(X9-Pin_4) -> Net-(X8-Pin_5)
- R37 pad 2: Net-(X12-Pin_3) -> Net-(X10-Pin_4)
- R42 pad 1: Net-(X12-Pin_4) -> Net-(X10-Pin_5)
- R52 pad 2: Net-(X14-Pin_3) (its old number) -> Net-(X11-Pin_4)
- R57 pad 1: Net-(X14-Pin_4) -> Net-(X11-Pin_5)
- R6 pad 1: Net-(X7-Pin_4) -> Net-(X7-Pin_5)
- R67 pad 2: Net-(X16-Pin_3) -> Net-(X12-Pin_4)
- R72 pad 1: Net-(X16-Pin_4) -> Net-(X12-Pin_5)
- R82 pad 2: Net-(X18-Pin_3) -> Net-(X13-Pin_4)
- R87 pad 1: Net-(X18-Pin_4) -> Net-(X13-Pin_5)
- X10 pad 3: Net-(X12-Pin_3) -> unconnected-(X10-Pin_3-Pad3)
- X10 pad 4: Net-(X12-Pin_4) -> Net-(X10-Pin_4)
- X10 pad 5: Net-(Q28-C) -> Net-(X10-Pin_5)
- X10 pad 6: Net-(Q29-C) -> Net-(Q28-C)
- X11 pad 3: Net-(X14-Pin_3) (its old number) -> unconnected-(X11-Pin_3-Pad3)
- X11 pad 4: Net-(X14-Pin_4) -> Net-(X11-Pin_4)
- X11 pad 5: Net-(Q39-C) -> Net-(X11-Pin_5)
- X11 pad 6: Net-(Q40-C) -> Net-(Q39-C)
- X12 pad 3: Net-(X16-Pin_3) -> unconnected-(X12-Pin_3-Pad3)
- X12 pad 4: Net-(X16-Pin_4) -> Net-(X12-Pin_4)
- X12 pad 5: Net-(Q50-C) -> Net-(X12-Pin_5)
- X12 pad 6: Net-(Q51-C) -> Net-(Q50-C)
- X13 pad 3: Net-(X18-Pin_3) -> unconnected-(X13-Pin_3-Pad3)
- X13 pad 4: Net-(X18-Pin_4) -> Net-(X13-Pin_4)
- X13 pad 5: Net-(Q61-C) -> Net-(X13-Pin_5)
- X13 pad 6: Net-(Q62-C) -> Net-(Q61-C)
- X7 pad 3: Net-(X7-Pin_3) -> unconnected-(X7-Pin_3-Pad3)
- X7 pad 5: Net-(Q4-C) -> Net-(X7-Pin_5)
- X7 pad 6: Net-(Q5-C) -> Net-(Q4-C)
- X8 pad 1: Net-(Q6-C) -> Net-(Q12-C)
- X8 pad 2: Net-(Q7-C) -> Net-(Q13-C)
- X8 pad 3: Net-(Q8-C) -> unconnected-(X8-Pin_3-Pad3)
- X8 pad 4: Net-(Q9-C) -> Net-(X8-Pin_4)
- X8 pad 5: Net-(Q10-C) -> Net-(X8-Pin_5)
- X8 pad 6: Net-(Q11-C) -> Net-(Q15-C)
Routing:
- net /Tube_1-2/GND: track 1995.7 -> 2051.9 mm, vias 22 -> 21
- net /Tube_1-2/SDA: track 310.9 -> 334.8 mm
- net /Tube_1-2/SCL: track 305.9 -> 326.2 mm
- net /Tube_1-2/3V3: track 956.3 -> 976.0 mm, vias 10 -> 9
- net Net-(X13-Pin_5): track 0.00 -> 13.8 mm
- net Net-(X11-Pin_5): track 0.00 -> 13.8 mm
- net Net-(X8-Pin_5): track 0.00 -> 13.8 mm
- net Net-(U1-ON/OFF): track 2.54 -> 16.3 mm
- net Net-(X7-Pin_5): track 0.00 -> 11.2 mm
- net Net-(X10-Pin_5): track 0.00 -> 11.2 mm
- net Net-(X12-Pin_5): track 0.00 -> 11.2 mm
- net Net-(X15-Pin_2): track 49.3 -> 39.2 mm
- net Net-(X15-Pin_1): track 44.2 -> 34.1 mm
- net Net-(R72-Pad2): track 10.2 -> 2.54 mm
- net Net-(X18-Pin_4): track 7.62 -> 0.00 mm
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Other:
- board size 307.3 x 144.8 mm -> 317.5 x 137.2 mm
- board text removed: "V2.3"
