File: NTC/Main.kicad_pcb (KiCad board)
At the start: 2 copper layers, 317.5 x 137.2 mm, 247 parts, among them Q1 MPSA42, Q10 MPSA42, Q11 MPSA42, Q12 MPSA42, Q13 MPSA42, Q14 MPSA42, Q15 MPSA42, Q16 MPSA42, Q17 MPSA42, Q18 MPSA42, Q19 MPSA42, Q2 MPSA42, Q20 MPSA42, Q21 MPSA42, Q22 MPSA42, Q23 MPSA42, Q24 MPSA42, Q25 MPSA42, Q26 MPSA42, Q27 MPSA42, Q28 MPSA42, Q29 MPSA42, Q3 MPSA42, Q30 MPSA42, Q31 MPSA42, Q32 MPSA42, Q33 MPSA42, Q34 MPSA42, Q35 MPSA42, Q36 MPSA42, Q37 MPSA42, Q38 MPSA42, Q39 MPSA42, Q4 MPSA42, Q40 MPSA42, Q41 MPSA42, Q42 MPSA42, Q43 MPSA42, Q44 MPSA42, Q45 MPSA42, Q46 MPSA42, Q47 MPSA42, Q48 MPSA42, Q49 MPSA42, Q5 MPSA42, Q50 MPSA42, Q51 MPSA42, Q52 MPSA42, Q53 MPSA42, Q54 MPSA42, Q55 MPSA42, Q56 MPSA42, Q57 MPSA42, Q58 MPSA42, Q59 MPSA42, Q6 MPSA42, Q60 MPSA42, Q61 MPSA42, Q62 MPSA42, Q63 MPSA42, Q64 MPSA42, Q65 MPSA42, Q66 MPSA42, Q67 MPSA42, Q68 MPSA42, Q69 MPSA42, Q7 MPSA42, Q70 MPSA42, Q8 MPSA42, Q9 MPSA42, U1 TDN_5-0911WISM, U2 R-78E5.0-1.0, X1 Barrel_Jack_Switch, X10 Conn_01x06_Socket, X11 Conn_01x06_Socket, X12 Conn_01x06_Socket, X13 Conn_01x06_Socket, X14 Conn_01x04_Socket, X15 Conn_01x04_Socket, X2.1 Conn_01x01_Pin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

Commit message: Added GPS
Parts:
- removed E20, E21: ~, Nixie:SingleHole
- added E31: ~, Nixie:SingleHole, F.Cu at (284.5, 55.9)
- added E32: ~, Nixie:SingleHole, F.Cu at (281.9, 55.9)
- added E33: ~, Nixie:SingleHole, F.Cu at (276.9, 162.6)
- added E34: ~, Nixie:SingleHole, F.Cu at (279.4, 162.6)
- added E35: ~, Nixie:SingleHole, F.Cu at (363.2, 162.6)
- added Q71: MPSA42, Nixie:MPSA-42, F.Cu at (63.5, 160.0)
- added R103: R, Nixie:Resistor-a, F.Cu at (66.0, 170.2)
- added X16.1: Conn_01x01_Pin, Nixie:Pin_D1.0mm_L10.0mm, F.Cu at (61.0, 175.3)
- added X16.2: Conn_01x01_Pin, Nixie:Pin_D1.0mm_L10.0mm, F.Cu at (66.0, 175.3)
- added X17: Conn_01x04_Socket, Nixie:Pinbar_1-4-f-c, F.Cu at (320.0, 50.8)
- added X18: Conn_01x04_Socket, Nixie:Pinbar_1-4-f-d, F.Cu at (152.4, 55.9)
- added X2.3: Conn_01x01_Pin, Nixie:Pin_D1.0mm_L10.0mm, F.Cu at (55.9, 129.5)
- moved E26 201.9 mm to (94.0, 129.5)
- moved E30 194.4 mm to (200.7, 55.9)
- moved E27 188.1 mm to (129.5, 162.6)
- moved E25 134.1 mm to (94.0, 137.2)
- moved E24 107.0 mm to (94.0, 142.2)
- moved E23 104.3 mm to (94.0, 144.8)
- moved E29 79.8 mm to (198.1, 149.9)
- moved E28 79.8 mm to (200.7, 149.9)
- moved E22 38.7 mm to (94.0, 147.3)
- moved E15 32.3 mm to (71.1, 177.8)
- moved E14 29.0 mm to (71.1, 175.3)
- moved E16 20.3 mm to (94.0, 172.7)
- moved E18 12.7 mm to (94.0, 157.5)
- moved E19 12.7 mm to (94.0, 154.9)
- moved E17 10.2 mm to (94.0, 160.0)
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Connections:
- E10 pad 1: Net-(X6-Pin_16) -> Net-(X6-Pin_14)
- E11 pad 1: Net-(X6-Pin_17) -> Net-(X6-Pin_15)
- E12 pad 1: Net-(X6-Pin_19) -> Net-(X6-Pin_16)
- E13 pad 1: Net-(X6-Pin_20) -> Net-(X6-Pin_18)
- E14 pad 1: Net-(X6-Pin_29) -> Net-(X6-Pin_19)
- E15 pad 1: Net-(X6-Pin_30) -> Net-(X6-Pin_20)
- E16 pad 1: Net-(X6-Pin_31) -> Net-(X6-Pin_23)
- E17 pad 1: Net-(X6-Pin_32) -> Net-(X6-Pin_28)
- E18 pad 1: Net-(X6-Pin_34) -> Net-(X6-Pin_29)
- E19 pad 1: Net-(X6-Pin_35) -> Net-(X6-Pin_30)
- E22 pad 1: Net-(A1-INT) -> Net-(X6-Pin_33)
- E23 pad 1: Net-(A2-INTA) -> Net-(X6-Pin_34)
- E24 pad 1: Net-(A2-INTB) -> Net-(X6-Pin_35)
- E25 pad 1: Net-(A3-INT) -> Net-(X6-Pin_37)
- E26 pad 1: Net-(A4-INTA) -> Net-(X6-Pin_40)
- E27 pad 1: Net-(A4-INTB) -> Net-(A1-INT)
- E28 pad 1: Net-(A5-INTA) -> Net-(A2-INTB)
- E29 pad 1: Net-(A5-INTB) -> Net-(A2-INTA)
- E3 pad 1: Net-(X6-Pin_7) -> Net-(X6-Pin_3)
- E30 pad 1: Net-(A6-INT) -> Net-(A3-INT)
- E4 pad 1: Net-(X6-Pin_9) -> Net-(X6-Pin_7)
- E5 pad 1: Net-(X6-Pin_10) -> Net-(X6-Pin_8)
- E6 pad 1: Net-(X6-Pin_11) -> Net-(X6-Pin_9)
- E7 pad 1: Net-(X6-Pin_12) -> Net-(X6-Pin_10)
- E8 pad 1: Net-(X6-Pin_14) -> Net-(X6-Pin_11)
- E9 pad 1: Net-(X6-Pin_15) -> Net-(X6-Pin_12)
- X3.1 pad 1: Net-(U1-+VIN) -> Net-(X2.3-Pin_1)
- X6 pad 13: unconnected-(X6-Pin_13-Pad13) -> Net-(Q71-E)
- X6 pad 18: unconnected-(X6-Pin_18-Pad18) -> Net-(X6-Pin_18)
- X6 pad 21: Net-(X15-Pin_2) -> Net-(X18-Pin_2)
- X6 pad 22: Net-(X15-Pin_1) -> Net-(X18-Pin_3)
- X6 pad 23: unconnected-(X6-Pin_23-Pad23) -> Net-(X6-Pin_23)
- X6 pad 24: /Tube_1-2/SDA -> Net-(X15-Pin_2)
- X6 pad 25: /Tube_1-2/SCL -> Net-(X15-Pin_1)
- X6 pad 26: /Tube_3-4/SDA -> /Tube_1-2/SDA
- X6 pad 27: /Tube_3-4/SCL -> /Tube_1-2/SCL
- X6 pad 28: unconnected-(X6-Pin_28-Pad28) -> Net-(X6-Pin_28)
- X6 pad 3: unconnected-(X6-Pin_3-Pad3) -> Net-(X6-Pin_3)
- X6 pad 31: Net-(X6-Pin_31) -> /Tube_3-4/SDA
- X6 pad 32: Net-(X6-Pin_32) -> /Tube_3-4/SCL
- X6 pad 33: unconnected-(X6-Pin_33-Pad33) -> Net-(X6-Pin_33)
- X6 pad 8: unconnected-(X6-Pin_8-Pad8) -> Net-(X6-Pin_8)
Routing:
- net Net-(X18-Pin_2): track 0.00 -> 192.3 mm, vias 0 -> 2
- net Net-(X18-Pin_3): track 0.00 -> 176.5 mm, vias 0 -> 2
- net /Tube_1-2/GND: track 2051.9 -> 1960.8 mm
- net /Tube_3-4/SCL: track 403.9 -> 349.6 mm, vias 2 -> 1
- net /Tube_3-4/SDA: track 411.5 -> 357.3 mm, vias 4 -> 3
- net Net-(X2.3-Pin_1): track 0.00 -> 44.8 mm
- net /Tube_1-2/3V3: track 976.0 -> 937.1 mm, vias 9 -> 10
- net Net-(U1-+VIN): track 54.6 -> 89.1 mm, vias 0 -> 1
- net /Tube_1-2/170V: track 306.9 -> 278.1 mm
- net /Tube_1-2/SCL: track 326.2 -> 309.0 mm, vias 0 -> 1
- net /Tube_1-2/SDA: track 334.8 -> 323.2 mm, vias 4 -> 5
- net Net-(Q71-C): track 0.00 -> 11.2 mm
- net Net-(Q71-E): track 0.00 -> 10.2 mm
- net Net-(X6-Pin_17): track 2.54 -> 7.62 mm
- net Net-(X15-Pin_2): track 39.2 -> 43.8 mm
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Other:
- outline, holes or cut-outs redrawn
- board text added: "BUZZ"
- board text added: "DCF77"

Commit message: Added GPS
Parts:
- removed E13, E22, E3, E5: ~, Nixie:SingleHole
- removed the REF** at (212.1, 166.4)
- removed the REF** at (237.5, 166.4)
- added E20: ~, Nixie:SingleHole, F.Cu at (94.0, 160.0)
- added E21: ~, Nixie:SingleHole, F.Cu at (94.0, 172.7)
- added REF**: Hole_M3, Nixie:Hole_M3, F.Cu at (231.1, 165.1)
- added REF**: Hole_M3, Nixie:Hole_M3, F.Cu at (246.4, 58.4)
- moved E16 38.1 mm to (94.0, 134.6)
- moved E17 12.7 mm to (94.0, 147.3)
- moved X18 2.54 mm to (154.9, 55.9)
Connections:
- E16 pad 1: Net-(X6-Pin_23) -> /Tube_1-2/GND
- E17 pad 1: Net-(X6-Pin_28) -> /Tube_1-2/GND
- Q71 pad 1: Net-(Q71-E) -> /Tube_1-2/GND
- X18 pad 1: /Tube_1-2/3V3 -> /Tube_1-2/GND
- X18 pad 4: /Tube_1-2/GND -> /Tube_1-2/3V3
- X6 pad 13: Net-(Q71-E) -> /Tube_1-2/GND
- X6 pad 18: Net-(X6-Pin_18) -> /Tube_1-2/GND
- X6 pad 21: Net-(X18-Pin_2) -> Net-(X18-Pin_3)
- X6 pad 22: Net-(X18-Pin_3) -> Net-(X18-Pin_2)
- X6 pad 23: Net-(X6-Pin_23) -> /Tube_1-2/GND
- X6 pad 28: Net-(X6-Pin_28) -> /Tube_1-2/GND
- X6 pad 3: Net-(X6-Pin_3) -> /Tube_1-2/GND
- X6 pad 33: Net-(X6-Pin_33) -> /Tube_1-2/GND
- X6 pad 8: Net-(X6-Pin_8) -> /Tube_1-2/GND
Routing:
- net /Tube_1-2/GND: track 1960.8 -> 2071.5 mm, vias 21 -> 20
- net Net-(X18-Pin_2): track 192.3 -> 178.0 mm
- net Net-(Q71-E): track 10.2 -> 0.00 mm
- net /Tube_1-2/3V3: track 937.1 -> 947.2 mm, vias 10 -> 9
- net Net-(X6-Pin_33): track 2.54 -> 0.00 mm
- net Net-(X6-Pin_28): track 2.54 -> 0.00 mm
- net Net-(X6-Pin_23): track 2.54 -> 0.00 mm
- net Net-(X6-Pin_8): track 2.54 -> 0.00 mm
- net Net-(X6-Pin_3): track 2.54 -> 0.00 mm
- net Net-(X6-Pin_18): track 2.54 -> 0.00 mm
- net Net-(X18-Pin_3): track 176.5 -> 178.0 mm
- net /Tube_1-2/SDA: vias 5 -> 4
Other:
- board text added: "IN1"
- board text added: "IN2"
- board text removed: "DCF77"
- board text removed: "IN"
