File: NTC/Tube_5-6.kicad_sch (KiCad schematic)
At the start: 70 parts, among them Q47 MPSA42, Q48 MPSA42, Q49 MPSA42, Q50 MPSA42, Q51 MPSA42, Q52 MPSA42, Q53 MPSA42, Q54 MPSA42, Q55 MPSA42, Q56 MPSA42, Q57 MPSA42, Q58 MPSA42, Q59 MPSA42, Q60 MPSA42, Q61 MPSA42, Q62 MPSA42, Q63 MPSA42, Q64 MPSA42, Q65 MPSA42, Q66 MPSA42, Q67 MPSA42, Q68 MPSA42, Q69 MPSA42, Q70 MPSA42, X16 Conn_01x06_Socket, X17 Conn_01x06_Socket, X18 Conn_01x06_Socket, X19 Conn_01x06_Socket, X20 Conn_01x04_Socket

Commit message: Changed to 14pin socket
Parts:
- removed X17, X19: Conn_01x06_Socket, Nixie:Pinbar_1-6-f-b, symbol Connector:Conn_01x06_Socket
- A5: footprint Package_DIP:DIP-28_W7.62mm -> Nixie:DIP-28_IC+Socket
- A6: footprint Package_DIP:DIP-18_W7.62mm -> Nixie:DIP-18_IC+Socket
- Q47, Q48, Q49, Q50, Q51, Q52, Q53, Q54, Q55, Q56, Q57, Q58, Q59, Q60, Q61, Q62, Q63, Q64, Q65, Q66, Q67, Q68, Q69, Q70: footprint Package_TO_SOT_THT:TO-92_Inline -> Nixie:MPSA-42
- X12: renamed from X16; footprint Nixie:Pinbar_1-6-f-a -> Nixie:Pinbar_4-14-f; symbol Connector:Conn_01x06_Socket -> Connector:Conn_01x14_Socket
- X13: renamed from X18; footprint Nixie:Pinbar_1-6-f-a -> Nixie:Pinbar_4-14-f; symbol Connector:Conn_01x06_Socket -> Connector:Conn_01x14_Socket
- renumbered X20 to X14
Connections:
- net at Q68.3 (C): now also X13.14 (Pin_14)
- net at R82.2: now also X13.4 (Pin_4); no longer X13.3 (Pin_3)
- net at Q56.3 (C): now also X12.13 (Pin_13)
- net at Q66.3 (C): now also X13.12 (Pin_12)
- net at Q50.3 (C): now also X12.6 (Pin_6); no longer X12.5 (Pin_5)
- net at Q52.3 (C): now also X12.8 (Pin_8)
- net at X12.3 (Pin_3): no longer R67.2
- net at X12.4 (Pin_4): now also R67.2; no longer R72.1
- net at Q51.3 (C): now also X12.7 (Pin_7); no longer X12.6 (Pin_6)
- net at Q57.3 (C): now also X12.14 (Pin_14)
- net at Q64.3 (C): now also X13.9 (Pin_9)
- net at R87.1: now also X13.5 (Pin_5); no longer X13.4 (Pin_4)
- net at Q61.3 (C): now also X13.6 (Pin_6); no longer X13.5 (Pin_5)
- net at Q62.3 (C): now also X13.7 (Pin_7); no longer X13.6 (Pin_6)
- net at Q67.3 (C): now also X13.13 (Pin_13)
- net at Q53.3 (C): now also X12.9 (Pin_9)
- net at Q54.3 (C): now also X12.10 (Pin_10)
- net at Q55.3 (C): now also X12.12 (Pin_12)
- net at Q65.3 (C): now also X13.10 (Pin_10)
- net at Q63.3 (C): now also X13.8 (Pin_8)
- new net: R72.1, X12.5 (Pin_5)
- no-connect marks 0 -> 4

Commit message: Added GPS
Parts:
- renumbered E29 to E33, E28 to E34, E30 to E35
Changed lines of the file:
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@@
 		(dnp no)
 		(fields_autoplaced yes)
-		(property "Reference" "E29"
+		(property "Reference" "E33"
 			(at 40.64 45.72 0)
 			(effects
@@
 			(project ""
 				(path "/ecf22f8e-0676-4495-9357-338c1fd23f92/ab4ab2d1-bcec-4364-97ac-9f7855117a69"
-					(reference "E29")
+					(reference "E33")
 					(unit 1)
 				)
@@
 		(dnp no)
 		(fields_autoplaced yes)
-		(property "Reference" "E28"
+		(property "Reference" "E34"
 			(at 40.64 48.26 0)
 			(effects
@@
 			(project ""
 				(path "/ecf22f8e-0676-4495-9357-338c1fd23f92/ab4ab2d1-bcec-4364-97ac-9f7855117a69"
-					(reference "E28")
+					(reference "E34")
 					(unit 1)
 				)
@@
 		(dnp no)
 		(fields_autoplaced yes)
-		(property "Reference" "E30"
+		(property "Reference" "E35"
 			(at 40.64 132.08 0)
 			(effects
@@
 			(project ""
 				(path "/ecf22f8e-0676-4495-9357-338c1fd23f92/ab4ab2d1-bcec-4364-97ac-9f7855117a69"
-					(reference "E30")
+					(reference "E35")
 					(unit 1)
 				)
